File: hardware/macropad_v1.0/macropad_v1.0.kicad_pcb (KiCad board)
At the start: 2 copper layers, 66.7 x 81 mm, 50 parts, among them J1 USB_C_Receptacle_USB2.0_14P, SW1 SW_Push, SW2 Rotary Encoder, SW3 Rotary Encoder, U1 USBLC6-2SC6, U2 STM32F072C8T6, U3 XC6206PxxxMR

Commit message: Finalized Silkscreen
-Made sure references weren't interfering with pads/vias/etc.

-Added BP logo to front

-Moved trace to decap slightly so that it wasn't interfering with mcu silkscreen

-Added BOOT0 and ON designators to boot button and on diode

-Added name and designed by to back silkscreen
Parts:
- added G***: LOGO, LOGO, F.Cu at (200.0, 22.0)
- moved C1 0.45 mm to (214.9, 61.2)
Other:
- board text added: "BOOT0 ▼"
- board text added: "Designed by Ben Pegg"
- board text added: "ON▼"
- board text added: "PARpad v1.0"
